File: Hardware/Production/expLoRaBLE Thing Plus-Panel_v11.brd (EAGLE design)
At the start: 130 x 206.5 mm, 2151 parts, among them J10 CORTEX_DEBUG, J100 USB Female Type C Connector, J101 CORTEX_DEBUG, J102 QWIIC_RIGHT_ANGLE, J105 U.FL, J11 QWIIC_RIGHT_ANGLE, J14 U.FL, J16 USB Female Type C Connector, J17 CORTEX_DEBUG, J18 QWIIC_RIGHT_ANGLE, J2 CORTEX_DEBUG, J21 U.FL, J23 USB Female Type C Connector, J24 CORTEX_DEBUG, J25 QWIIC_RIGHT_ANGLE, J28 U.FL, J30 USB Female Type C Connector, J31 CORTEX_DEBUG, J32 QWIIC_RIGHT_ANGLE, J35 U.FL, J37 USB Female Type C Connector, J38 CORTEX_DEBUG, J39 QWIIC_RIGHT_ANGLE, J42 U.FL, J44 USB Female Type C Connector, J45 CORTEX_DEBUG, J46 QWIIC_RIGHT_ANGLE, J49 U.FL, J5 USB Female Type C Connector, J51 USB Female Type C Connector, J52 CORTEX_DEBUG, J53 QWIIC_RIGHT_ANGLE, J56 U.FL, J58 USB Female Type C Connector, J59 CORTEX_DEBUG, J6 QWIIC_RIGHT_ANGLE, J60 QWIIC_RIGHT_ANGLE, J63 U.FL, J65 USB Female Type C Connector, J66 CORTEX_DEBUG, J67 QWIIC_RIGHT_ANGLE, J70 U.FL, J72 USB Female Type C Connector, J73 CORTEX_DEBUG, J74 QWIIC_RIGHT_ANGLE, J77 U.FL, J79 USB Female Type C Connector, J8 U.FL, J80 CORTEX_DEBUG, J81 QWIIC_RIGHT_ANGLE, J84 U.FL, J86 USB Female Type C Connector, J87 CORTEX_DEBUG, J88 QWIIC_RIGHT_ANGLE, J9 USB Female Type C Connector, J91 U.FL, J93 USB Female Type C Connector, J94 CORTEX_DEBUG, J95 QWIIC_RIGHT_ANGLE, J98 U.FL, U1 MCP73831, U10 DPX202700DT-4162A1, U11 MCP73831, U12 3.3V, U13 CH340E_MSOP10, U14 NM180100, U15 DPX202700DT-4162A1, U16 MCP73831, U17 3.3V, U18 CH340E_MSOP10, U19 NM180100, U2 3.3V, U20 DPX202700DT-4162A1, U21 MCP73831, U22 3.3V, U23 CH340E_MSOP10, U24 NM180100, U25 DPX202700DT-4162A1, U26 MCP73831, U27 3.3V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

Commit message: v11 production panel BRD and gerbers
Parts:
- added C226: 15pF, SparkFun-Capacitors:0603
- added C227: 10nF, SparkFun-Capacitors:0603
- added C228, C229, C239, C240: 0.1uF, SparkFun-Capacitors:0603
- added C230: 10uF, SparkFun-Capacitors:0603
- added C231, C235, C236: 1.0uF, SparkFun-Capacitors:0603
- added C232: 1nF, SparkFun-Capacitors:0603
- added C233, C234: 4.7uF, SparkFun-Capacitors:0603
- added C237: 47pF, SparkFun-Capacitors:0603
- added C238: 10pF, SparkFun-Capacitors:0603
- added R151, R153, R156, R158, R161, R162, R164: 1k, SparkFun-Resistors:0603
- added R152, R163: 2.0k, SparkFun-Resistors:0603
- added R154, R165: 220k, SparkFun-Resistors:0603
- added R155: 10k, SparkFun-Resistors:0603
- added R157, R159: 5.1k, SparkFun-Resistors:0603
- added R160: 100k, SparkFun-Resistors:0603
- C100, C144, C159, C160, C175, C69, C84, C85: value 4.7uF -> 0.1uF
- C101, C112, C116, C117, C127, C132, C176, C191, C192, C207, C37, C52: value 1.0uF -> 0.1uF
- C102, C22, C86: value 1.0uF -> 10uF
- C103, C28, C43: value 47pF -> 1.0uF
- C104: value 10pF -> 1nF
- C105, C154, C169, C170, C185, C90: value 0.1uF -> 4.7uF
- C106, C121, C122, C137: value 15pF -> 4.7uF
- C107, C151, C167, C76, C91, C92: value 15pF -> 1.0uF
- C108, C123, C183: value 10nF -> 1.0uF
- C109, C125, C45: value 0.1uF -> 47pF
- C110, C30, C94: value 0.1uF -> 10pF
- C111, C21, C36, C96: value 10uF -> 0.1uF
- C113, C98: value 1nF -> 15pF
- C114, C129, C130, C145: value 4.7uF -> 15pF
- C115, C99: value 4.7uF -> 10nF
- C118: value 47pF -> 10uF
- C119, C44, C59: value 10pF -> 1.0uF
- C120, C184, C200: value 0.1uF -> 1nF
- C124, C135, C139, C140, C155, C199, C215, C60, C75: value 0.1uF -> 1.0uF
- C126: value 10uF -> 10pF
- C128, C143, C53, C68: value 1nF -> 0.1uF
- C13, C181, C196, C197, C212, C31, C32, C47: value 15pF -> 0.1uF
- C131, C147, C67: value 1.0uF -> 10nF
- C133, C148, C208, C223: value 47pF -> 0.1uF
- C134: value 10pF -> 10uF
- C136, C152: value 15pF -> 1nF
- C138, C153: value 10nF -> 4.7uF
- C141: value 10uF -> 47pF
- C142, C206, C222: value 1.0uF -> 10pF
- C146, C161, C162, C177, C82, C97: value 1.0uF -> 15pF
- C149, C164, C224: value 10pF -> 0.1uF
- C150, C214: value 0.1uF -> 10uF
- C156, C171: value 10uF -> 1.0uF
- C157, C221: value 1.0uF -> 47pF
- C158: value 1nF -> 10pF
- C163: value 47pF -> 10nF
- C166, C182: value 15pF -> 10uF
- C168: value 10nF -> 1nF
- C173: value 1nF -> 47pF
- C174, C190: value 4.7uF -> 10pF
- C178, C193: value 47pF -> 15pF
- C179: value 10pF -> 10nF
- C18, C33: value 10nF -> 15pF
- C186, C201: value 10uF -> 4.7uF
- C188, C203, C23: value 1nF -> 1.0uF
- C189, C205: value 4.7uF -> 47pF
- C19, C195, C35: value 0.1uF -> 10nF
- C194, C209: value 10pF -> 15pF
- C198: value 10nF -> 10uF
- C202, C217, C26, C41, C42, C57: value 1.0uF -> 4.7uF
- C204, C219, C220, C39, C55: value 4.7uF -> 1.0uF
- C210, C225, C34, C49, C50, C65: value 0.1uF -> 15pF
- C211: value 15pF -> 10nF
- C213, C48, C63: value 10nF -> 0.1uF
- C216: value 10uF -> 1nF
- C218: value 1nF -> 4.7uF
- C24, C40: value 4.7uF -> 1nF
- C29: value 10pF -> 47pF
- C38: value 1nF -> 10uF
- C46, C62: value 15pF -> 10pF
- C51: value 10uF -> 10nF
- C54, C70: value 4.7uF -> 10uF
- C56, C72: value 1.0uF -> 1nF
- C58, C73: value 47pF -> 4.7uF
- C61, C77: value 15pF -> 47pF
- C66, C81: value 10uF -> 15pF
- C74, C89: value 10pF -> 4.7uF
- C78: value 10nF -> 10pF
- C83: value 1nF -> 10nF
- C88: value 47pF -> 1nF
- C93: value 10nF -> 47pF
- J102, J11, J18, J25, J32, J39, J46, J53, J6, J60, J67, J74, J81, J88, J95: value QWIIC_RIGHT_ANGLE -> QWIIC_RA
- R10, R110, R132, R22, R44, R77, R88: value 1k -> 220k
- R100, R122, R144, R34, R67, R78: value 1k -> 10k
- R101, R131, R21, R41, R51, R81: value 10k -> 1k
- R102, R104, R124, R137, R14, R148, R27, R38, R47, R58, R60, R80, R82: value 1k -> 5.1k
- R103, R123, R125, R13, R145, R15, R35, R43, R63, R65, R73, R85, R95: value 5.1k -> 1k
- R105, R83: value 5.1k -> 100k
- R106, R136, R26, R46, R76, R96: value 100k -> 1k
- R108, R130, R20, R42, R64, R97: value 1k -> 2.0k
- R109, R129, R139, R19, R29, R59, R79: value 2.0k -> 1k
- R121: value 10k -> 220k
- R126, R146, R16, R36: value 100k -> 5.1k
- R127, R138, R17, R28, R50, R72, R94: value 1k -> 100k
- R133, R23, R45: value 5.1k -> 10k
- R141, R31: value 10k -> 2.0k
- R143, R33, R55: value 5.1k -> 220k
- R149, R39: value 2.0k -> 100k
- R49, R69: value 2.0k -> 5.1k
- R53, R75: value 5.1k -> 2.0k
- R56: value 100k -> 10k
- R61: value 10k -> 100k
- R66: value 100k -> 220k
- R71, R91: value 10k -> 5.1k
- R86: value 100k -> 2.0k
- R89: value 2.0k -> 10k
- R99: value 2.0k -> 220k
- RTS, RTS1, RTS10, RTS11, RTS12, RTS13, RTS14, RTS2, RTS3, RTS4, RTS5, RTS6, RTS7, RTS8, RTS9: value JUMPER-SMT_2_NO_SILK -> JUMPER-SMT_2_NC_TRACE_SILK; device SparkFun-Jumpers:SMT-JUMPER_2_NO_SILK -> SparkFun-Jumpers:SMT-JUMPER_2_NC_TRACE_SILK
- moved C152 131.9 mm to (109.5, 78.5), turned to 180 degrees
- moved R102 125.7 mm to (106.9, 71.9)
- moved R104 123.4 mm to (105.4, 71.9)
- moved R110 122.6 mm to (112.3, 86.2)
- moved C159 122.2 mm to (109.1, 85.4), turned to 0 degrees
- moved C160 122.0 mm to (109.1, 87.1), turned to 0 degrees
- moved C155 120.9 mm to (108.8, 81.3)
- moved C76 118.2 mm to (107.3, 27.5), turned to 0 degrees
- moved C80 117.4 mm to (109.1, 25.6)
- moved C156 117.1 mm to (107.3, 88.9), turned to 0 degrees
- moved R108 116.3 mm to (101.6, 84.1), turned to 0 degrees
- moved C79 116.0 mm to (109.1, 23.9), turned to 0 degrees
- moved C151 114.0 mm to (111.5, 101.2), turned to 0 degrees
- moved R105 112.6 mm to (109.5, 77.0), turned to 180 degrees
- moved R55 110.9 mm to (112.3, 24.7), turned to 90 degrees
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Connections:
- new net BOOT: C13.2, R10.2, U3.J7
- new net BOOT1: C32.2, R22.2, U9.J7
- new net BOOT10: C176.2, R121.2, U54.J7
- new net BOOT11: C192.2, R132.2, U59.J7
- new net BOOT12: C208.2, R143.2, U64.J7
- new net BOOT13: C224.2, R154.2, U69.J7
- new net BOOT14: C240.2, R165.2, U74.J7
- new net BOOT2: C48.2, R33.2, U14.J7
- new net BOOT3: C64.2, R44.2, U19.J7
- new net BOOT4: C80.2, R55.2, U24.J7
- new net BOOT5: C96.2, R66.2, U29.J7
- new net BOOT6: C112.2, R77.2, U34.J7
- new net BOOT7: C128.2, R88.2, U39.J7
- new net BOOT8: C144.2, R99.2, U44.J7
- new net BOOT9: C160.2, R110.2, U49.J7
- net !RESET: now also C1.2; no longer RTS.2
- net !RESET1: now also C24.1, C31.2, R17.1; no longer C23.1, R16.1, RTS1.2
- net !RESET10: now also C168.1, C175.2, R116.1; no longer C158.1, R106.1, RTS10.2
- net !RESET11: now also C184.1, C191.2, R127.1; no longer C173.1, R116.1, RTS11.2
- net !RESET12: now also C200.1, C207.2, R138.1; no longer C188.1, R126.1, RTS12.2
- net !RESET13: now also C216.1, C223.2, R149.1; no longer C203.1, R136.1, RTS13.2
- net !RESET14: now also C232.1, C239.2, R160.1; no longer C218.1, R146.1, RTS14.2
- net !RESET2: now also C40.1, C47.2, R28.1; no longer C38.1, R26.1, RTS2.2
- net !RESET3: now also C56.1, C63.2, R39.1; no longer C53.1, R36.1, RTS3.2
- net !RESET4: now also C72.1, C79.2, R50.1; no longer C68.1, R46.1, RTS4.2
- net !RESET5: now also C88.1, C95.2, R61.1; no longer C83.1, R56.1, RTS5.2
- net !RESET6: now also C104.1, C111.2, R72.1; no longer C98.1, R66.1, RTS6.2
- net !RESET7: now also C120.1, C127.2, R83.1; no longer C113.1, R76.1, RTS7.2
- net !RESET8: now also C136.1, C143.2, R94.1; no longer C128.1, R86.1, RTS8.2
- net !RESET9: now also C152.1, C159.2, R105.1; no longer C143.1, R96.1, RTS9.2
- net !RTS: now also RTS.1; no longer C1.1
- net !RTS1: now also RTS1.1; no longer C30.1
- net !RTS10: now also RTS10.1; no longer C165.1
- net !RTS11: now also RTS11.1; no longer C180.1
- net !RTS12: now also RTS12.1; no longer C195.1
- net !RTS13: now also RTS13.1; no longer C210.1
- net !RTS14: now also RTS14.1; no longer C225.1
- net !RTS2: now also RTS2.1; no longer C45.1
- net !RTS3: now also RTS3.1; no longer C60.1
- net !RTS4: now also RTS4.1; no longer C75.1
- net !RTS5: now also RTS5.1; no longer C90.1
- net !RTS6: now also RTS6.1; no longer C105.1
- net !RTS7: now also RTS7.1; no longer C120.1
- net !RTS8: now also RTS8.1; no longer C135.1
- net !RTS9: now also RTS9.1; no longer C150.1
- net 3.3V1: now also C23.1, C28.1, R15.2, R18.2; no longer C18.1, C27.1, R14.2, R16.2
- net 3.3V10: now also C163.1, C164.1, C165.1, C166.1, C167.1, C172.1, R114.2, R116.2, R117.2; no longer C153.1, C154.1, C155.1, C156.1, C157.1, C162.1, R104.2, R106.2, R107.2
- net 3.3V11: now also C179.1, C180.1, C181.1, C182.1, C183.1, C188.1, R125.2, R127.2, R128.2; no longer C168.1, C169.1, C170.1, C171.1, C172.1, C177.1, R114.2, R116.2, R117.2
- net 3.3V12: now also C195.1, C196.1, C197.1, C198.1, C199.1, C204.1, R136.2, R138.2, R139.2; no longer C183.1, C184.1, C185.1, C186.1, C187.1, C192.1, R124.2, R126.2, R127.2
- net 3.3V13: now also C211.1, C212.1, C213.1, C214.1, C215.1, C220.1, R147.2, R149.2, R150.2; no longer C198.1, C199.1, C200.1, C201.1, C202.1, C207.1, R134.2, R136.2, R137.2
- net 3.3V14: now also C227.1, C228.1, C229.1, C230.1, C231.1, C236.1, R158.2, R160.2, R161.2; no longer C213.1, C214.1, C215.1, C216.1, C217.1, C222.1, R144.2, R146.2, R147.2
- net 3.3V2: now also C38.1, C39.1, C44.1, R28.2, R29.2; no longer C33.1, C34.1, C42.1, R24.2, R27.2
- net 3.3V3: now also C53.1, C54.1, C55.1, C60.1, R39.2, R40.2; no longer C48.1, C49.1, C50.1, C57.1, R34.2, R36.2
- net 3.3V4: now also C68.1, C69.1, C70.1, C71.1, C76.1, R48.2, R50.2, R51.2; no longer C63.1, C64.1, C65.1, C66.1, C72.1, R44.2, R46.2, R47.2
- net 3.3V5: now also C83.1, C84.1, C85.1, C86.1, C92.1, R59.2, R61.2, R62.2; no longer C78.1, C79.1, C80.1, C81.1, C82.1, R54.2, R56.2, R57.2
- net 3.3V6: now also C100.1, C101.1, C103.1, C108.1, C99.1, R70.2, R72.2, R73.2; no longer C93.1, C94.1, C95.1, C96.1, C97.1, R64.2, R66.2, R67.2
- net 3.3V7: now also C115.1, C116.1, C118.1, C119.1, C124.1, R81.2, R83.2, R84.2; no longer C108.1, C109.1, C110.1, C111.1, C112.1, R74.2, R76.2, R77.2
- net 3.3V8: now also C131.1, C133.1, C134.1, C135.1, C140.1, R92.2, R94.2, R95.2; no longer C123.1, C124.1, C125.1, C126.1, C127.1, R84.2, R86.2, R87.2
- net 3.3V9: now also C148.1, C149.1, C150.1, C151.1, C156.1, R103.2, R105.2, R106.2; no longer C138.1, C139.1, C140.1, C141.1, C142.1, R94.2, R96.2, R97.2
- net BT_RF1: now also C30.1; no longer C29.1
- net BT_RF10: now also C174.1; no longer C164.1
- net BT_RF11: now also C190.1; no longer C179.1
- net BT_RF12: now also C206.1; no longer C194.1
- net BT_RF13: now also C222.1; no longer C209.1
- net BT_RF14: now also C238.1; no longer C224.1
- net BT_RF2: now also C46.1; no longer C44.1
- net BT_RF3: now also C62.1; no longer C59.1
- net BT_RF4: now also C78.1; no longer C74.1
- net BT_RF5: now also C94.1; no longer C89.1
- net BT_RF6: now also C110.1; no longer C104.1
- net BT_RF7: now also C126.1; no longer C119.1
- net BT_RF8: now also C142.1; no longer C134.1
- net BT_RF9: now also C158.1; no longer C149.1
- net CC10: now also R49.2; no longer R45.2
- net CC11: now also R58.2; no longer R53.2
- net CC12: now also R60.2; no longer R55.2
- net CC13: now also R69.2; no longer R63.2
- net CC14: now also R71.2; no longer R65.2
- net CC15: now also R80.2; no longer R73.2
- net CC16: now also R82.2; no longer R75.2
- net CC17: now also R91.2; no longer R83.2
- net CC18: now also R93.2; no longer R85.2
- net CC19: now also R102.2; no longer R93.2
- net CC20: now also R104.2; no longer R95.2
- net CC21: now also R113.2; no longer R103.2
- net CC22: now also R115.2; no longer R105.2
- net CC23: now also R124.2; no longer R113.2
- net CC24: now also R126.2; no longer R115.2
- net CC25: now also R135.2; no longer R123.2
- net CC26: now also R137.2; no longer R125.2
- net CC27: now also R146.2; no longer R133.2
- net CC28: now also R148.2; no longer R135.2
- net CC29: now also R157.2; no longer R143.2
- net CC3: now also R14.2; no longer R13.2
- net CC30: now also R159.2; no longer R145.2
- net CC4: now also R16.2; no longer R15.2
- net CC5: now also R25.2; no longer R23.2
- net CC6: now also R27.2; no longer R25.2
- net CC7: now also R36.2; no longer R33.2
- net CC8: now also R38.2; no longer R35.2
- net CC9: now also R47.2; no longer R43.2
- net D10/SWCH: now also U3.J6; no longer U3.J3
- net D10/SWCH1: now also U9.J6; no longer U9.J3
- net D10/SWCH10: now also U54.J6; no longer U54.J3
- net D10/SWCH11: now also U59.J6; no longer U59.J3
- net D10/SWCH12: now also U64.J6; no longer U64.J3
- net D10/SWCH13: now also U69.J6; no longer U69.J3
- net D10/SWCH14: now also U74.J6; no longer U74.J3
- net D10/SWCH2: now also U14.J6; no longer U14.J3
- net D10/SWCH3: now also U19.J6; no longer U19.J3
- net D10/SWCH4: now also U24.J6; no longer U24.J3
- net D10/SWCH5: now also U29.J6; no longer U29.J3
- net D10/SWCH6: now also U34.J6; no longer U34.J3
- net D10/SWCH7: now also U39.J6; no longer U39.J3
- net D10/SWCH8: now also U44.J6; no longer U44.J3
- net D10/SWCH9: now also U49.J6; no longer U49.J3
- net EN10: now also R111.1; no longer R101.1
- net EN11: now also R122.1; no longer R111.1
- net EN12: now also R133.1; no longer R121.1
- net EN13: now also R144.1; no longer R131.1
- net EN14: now also R155.1; no longer R141.1
- net EN2: now also R23.1; no longer R21.1
- net EN3: now also R34.1; no longer R31.1
- net EN4: now also R45.1; no longer R41.1
- net EN5: now also R56.1; no longer R51.1
- net EN6: now also R67.1; no longer R61.1
- net EN7: now also R78.1; no longer R71.1
- net EN8: now also R89.1; no longer R81.1
- net EN9: now also R100.1; no longer R91.1
- net GND: now also R10.1
- net GND1: now also C18.1, C28.2, R14.1, R16.1, R20.1, R22.1; no longer C13.1, C18.2, R13.1, R15.1, R19.1
- net GND10: now also C161.1, C162.1, C163.2, C164.2, C165.2, C166.2, C167.2, C168.2, C169.2, C170.2, C171.2, C172.2, R113.1, R115.1, R119.1, R121.1; no longer C151.1, C152.1, C153.2, C154.2, C155.2, C156.2, C157.2, C158.2, C159.2, C160.2, C161.2, C162.2, R103.1, R105.1, R109.1
- net GND11: now also C177.1, C178.1, C179.2, C180.2, C181.2, C182.2, C183.2, C184.2, C185.2, C186.2, C187.2, C188.2, R124.1, R126.1, R130.1, R132.1; no longer C166.1, C167.1, C168.2, C169.2, C170.2, C171.2, C172.2, C173.2, C174.2, C175.2, C176.2, C177.2, R113.1, R115.1, R119.1
- net GND12: now also C193.1, C194.1, C195.2, C196.2, C197.2, C198.2, C199.2, C200.2, C201.2, C202.2, C203.2, C204.2, R135.1, R137.1, R141.1, R143.1; no longer C181.1, C182.1, C183.2, C184.2, C185.2, C186.2, C187.2, C188.2, C189.2, C190.2, C191.2, C192.2, R123.1, R125.1, R129.1
- net GND13: now also C209.1, C210.1, C211.2, C212.2, C213.2, C214.2, C215.2, C216.2, C217.2, C218.2, C219.2, C220.2, R146.1, R148.1, R152.1, R154.1; no longer C196.1, C197.1, C198.2, C199.2, C200.2, C201.2, C202.2, C203.2, C204.2, C205.2, C206.2, C207.2, R133.1, R135.1, R139.1
- net GND14: now also C225.1, C226.1, C227.2, C228.2, C229.2, C230.2, C231.2, C232.2, C233.2, C234.2, C235.2, C236.2, R157.1, R159.1, R163.1, R165.1; no longer C211.1, C212.1, C213.2, C214.2, C215.2, C216.2, C217.2, C218.2, C219.2, C220.2, C221.2, C222.2, R143.1, R145.1, R149.1
- net GND2: now also C33.1, C34.1, C43.2, C44.2, R27.1, R31.1, R33.1; no longer C31.1, C32.1, C33.2, C34.2, R23.1, R29.1
- net GND3: now also C49.1, C50.1, C58.2, C59.2, C60.2, R36.1, R38.1, R42.1, R44.1; no longer C46.1, C47.1, C48.2, C49.2, C50.2, R33.1, R35.1, R39.1
- net GND4: now also C65.1, C66.1, C73.2, C74.2, C75.2, C76.2, R47.1, R53.1, R55.1; no longer C61.1, C62.1, C63.2, C64.2, C65.2, C66.2, R43.1, R45.1
- net GND5: now also C81.1, C82.1, C88.2, C89.2, C90.2, C91.2, C92.2, R58.1, R60.1, R64.1, R66.1; no longer C76.1, C77.1, C78.2, C79.2, C80.2, C81.2, C82.2, R53.1, R55.1, R59.1
- net GND6: now also C103.2, C104.2, C105.2, C106.2, C107.2, C108.2, C97.1, C98.1, R71.1, R75.1, R77.1; no longer C91.1, C92.1, C93.2, C94.2, C95.2, C96.2, C97.2, C98.2, R63.1, R65.1
- net GND7: now also C113.1, C114.1, C118.2, C119.2, C120.2, C121.2, C122.2, C123.2, C124.2, R80.1, R82.1, R86.1, R88.1; no longer C106.1, C107.1, C108.2, C109.2, C110.2, C111.2, C112.2, C113.2, C114.2, R73.1, R75.1, R79.1
- net GND8: now also C129.1, C130.1, C133.2, C134.2, C135.2, C136.2, C137.2, C138.2, C139.2, C140.2, R91.1, R93.1, R97.1, R99.1; no longer C121.1, C122.1, C123.2, C124.2, C125.2, C126.2, C127.2, C128.2, C129.2, C130.2, R83.1, R85.1, R89.1
- net GND9: now also C145.1, C146.1, C148.2, C149.2, C150.2, C151.2, C152.2, C153.2, C154.2, C155.2, C156.2, R102.1, R104.1, R108.1, R110.1; no longer C136.1, C137.1, C138.2, C139.2, C140.2, C141.2, C142.2, C143.2, C144.2, C145.2, C146.2, R93.1, R95.1, R99.1
- net LORA_RF1: now also C29.1; no longer C28.1
- net LORA_RF10: now also C173.1; no longer C163.1
- net LORA_RF11: now also C189.1; no longer C178.1
- net LORA_RF12: now also C205.1; no longer C193.1
- net LORA_RF13: now also C221.1; no longer C208.1
- net LORA_RF14: now also C237.1; no longer C223.1
- net LORA_RF2: now also C45.1; no longer C43.1
- net LORA_RF3: now also C61.1; no longer C58.1
- net LORA_RF4: now also C77.1; no longer C73.1
- net LORA_RF5: now also C93.1; no longer C88.1
- net LORA_RF6: now also C109.1; no longer C103.1
- net LORA_RF7: now also C125.1; no longer C118.1
- net LORA_RF8: now also C141.1; no longer C133.1
- net LORA_RF9: now also C157.1; no longer C148.1
- net N$101: now also C110.2; no longer C104.2
- net N$102: now also C109.2; no longer C103.2
- net N$104: now also R68.2; no longer R62.2
- net N$105: now also C111.1, C112.1, RTS6.2; no longer C105.2, RTS6.1
- net N$106: now also R79.1; no longer R72.1
- net N$107: now also R86.2; no longer R79.2
- net N$108: now also R87.2; no longer R80.2
- net N$109: now also R87.1; no longer R80.1
- net N$110: now also C113.2; no longer C106.2
- net N$111: now also C114.2; no longer C107.2
- net N$112: now also R85.1; no longer R78.1
- net N$113: now also R84.1; no longer R77.1
- net N$114: now also R81.1; no longer R74.1
- net N$116: now also C126.2; no longer C119.2
- net N$117: now also C125.2; no longer C118.2
- net N$119: now also R79.2; no longer R72.2
- net N$120: now also C127.1, C128.1, RTS7.2; no longer C120.2, RTS7.1
- net N$121: now also R90.1; no longer R82.1
- net N$122: now also R97.2; no longer R89.2
- net N$123: now also R98.2; no longer R90.2
- net N$124: now also R98.1; no longer R90.1
- net N$125: now also C129.2; no longer C121.2
- net N$126: now also C130.2; no longer C122.2
- net N$127: now also R96.1; no longer R88.1
- net N$128: now also R95.1; no longer R87.1
- net N$129: now also R92.1; no longer R84.1
- net N$131: now also C142.2; no longer C134.2
- net N$132: now also C141.2; no longer C133.2
- net N$134: now also R90.2; no longer R82.2
- net N$135: now also C143.1, C144.1, RTS8.2; no longer C135.2, RTS8.1
- net N$136: now also R101.1; no longer R92.1
- net N$137: now also R108.2; no longer R99.2
- net N$138: now also R109.2; no longer R100.2
- net N$139: now also R109.1; no longer R100.1
- net N$140: now also C145.2; no longer C136.2
- net N$141: now also C146.2; no longer C137.2
- net N$142: now also R107.1; no longer R98.1
- net N$143: now also R106.1; no longer R97.1
- net N$144: now also R103.1; no longer R94.1
- net N$146: now also C158.2; no longer C149.2
- net N$147: now also C157.2; no longer C148.2
- net N$149: now also R101.2; no longer R92.2
- net N$15: now also C1.1, C13.1, RTS.2; no longer C1.2, RTS.1
- net N$150: now also C159.1, C160.1, RTS9.2; no longer C150.2, RTS9.1
- net N$151: now also R112.1; no longer R102.1
- net N$152: now also R119.2; no longer R109.2
- net N$153: now also R120.2; no longer R110.2
- net N$154: now also R120.1; no longer R110.1
- net N$155: now also C161.2; no longer C151.2
- net N$156: now also C162.2; no longer C152.2
- net N$157: now also R118.1; no longer R108.1
- net N$158: now also R117.1; no longer R107.1
- net N$159: now also R114.1; no longer R104.1
- net N$16: now also R13.1; no longer R10.1
- net N$161: now also C174.2; no longer C164.2
- net N$162: now also C173.2; no longer C163.2
- net N$164: now also R112.2; no longer R102.2
- net N$165: now also C175.1, C176.1, RTS10.2; no longer C165.2, RTS10.1
- net N$166: now also R123.1; no longer R112.1
- net N$167: now also R130.2; no longer R119.2
- net N$168: now also R131.2; no longer R120.2
- net N$169: now also R131.1; no longer R120.1
- net N$17: now also R20.2; no longer R19.2
- net N$170: now also C177.2; no longer C166.2
- net N$171: now also C178.2; no longer C167.2
- net N$172: now also R129.1; no longer R118.1
- net N$173: now also R128.1; no longer R117.1
- net N$174: now also R125.1; no longer R114.1
- net N$176: now also C190.2; no longer C179.2
- net N$177: now also C189.2; no longer C178.2
- net N$179: now also R123.2; no longer R112.2
- net N$18: now also R21.2; no longer R20.2
- net N$180: now also C191.1, C192.1, RTS11.2; no longer C180.2, RTS11.1
- net N$181: now also R134.1; no longer R122.1
- net N$182: now also R141.2; no longer R129.2
- net N$183: now also R142.2; no longer R130.2
- net N$184: now also R142.1; no longer R130.1
- net N$185: now also C193.2; no longer C181.2
- net N$186: now also C194.2; no longer C182.2
- net N$187: now also R140.1; no longer R128.1
- net N$188: now also R139.1; no longer R127.1
- net N$189: now also R136.1; no longer R124.1
- net N$19: now also R21.1; no longer R20.1
- net N$191: now also C206.2; no longer C194.2
- net N$192: now also C205.2; no longer C193.2
- net N$194: now also R134.2; no longer R122.2
- net N$195: now also C207.1, C208.1, RTS12.2; no longer C195.2, RTS12.1
- net N$196: now also R145.1; no longer R132.1
- net N$197: now also R152.2; no longer R139.2
- net N$198: now also R153.2; no longer R140.2
- net N$199: now also R153.1; no longer R140.1
- net N$20: now also C14.2; no longer C13.2
- net N$200: now also C209.2; no longer C196.2
- net N$201: now also C210.2; no longer C197.2
- net N$202: now also R151.1; no longer R138.1
- net N$203: now also R150.1; no longer R137.1
- net N$204: now also R147.1; no longer R134.1
- net N$206: now also C222.2; no longer C209.2
- net N$207: now also C221.2; no longer C208.2
- net N$209: now also R145.2; no longer R132.2
- net N$21: now also C18.2; no longer C14.2
- net N$210: now also C223.1, C224.1, RTS13.2; no longer C210.2, RTS13.1
- net N$211: now also R156.1; no longer R142.1
- net N$212: now also R163.2; no longer R149.2
- net N$213: now also R164.2; no longer R150.2
- net N$214: now also R164.1; no longer R150.1
- net N$215: now also C225.2; no longer C211.2
- net N$216: now also C226.2; no longer C212.2
- net N$217: now also R162.1; no longer R148.1
- net N$218: now also R161.1; no longer R147.1
- net N$219: now also R158.1; no longer R144.1
- net N$22: now also R19.1; no longer R18.1
- net N$221: now also C238.2; no longer C224.2
- net N$222: now also C237.2; no longer C223.2
- net N$224: now also R156.2; no longer R142.2
- net N$225: now also C239.1, C240.1, RTS14.2; no longer C225.2, RTS14.1
- net N$23: now also R18.1; no longer R17.1
- net N$24: now also R15.1; no longer R14.1
- net N$26: now also C30.2; no longer C29.2
- net N$27: now also C29.2; no longer C28.2
- net N$29: now also R13.2; no longer R10.2
- net N$30: now also C31.1, C32.1, RTS1.2; no longer C30.2, RTS1.1
- net N$31: now also R24.1; no longer R22.1
- net N$32: now also R31.2; no longer R29.2
- net N$33: now also R32.2; no longer R30.2
- net N$34: now also R32.1; no longer R30.1
- net N$35: now also C33.2; no longer C31.2
- net N$36: now also C34.2; no longer C32.2
- net N$37: now also R30.1; no longer R28.1
- net N$38: now also R29.1; no longer R27.1
- net N$39: now also R26.1; no longer R24.1
- net N$41: now also C46.2; no longer C44.2
- net N$42: now also C45.2; no longer C43.2
- net N$44: now also R24.2; no longer R22.2
- net N$45: now also C47.1, C48.1, RTS2.2; no longer C45.2, RTS2.1
- net N$46: now also R35.1; no longer R32.1
- net N$47: now also R42.2; no longer R39.2
- net N$48: now also R43.2; no longer R40.2
- net N$49: now also R43.1; no longer R40.1
- net N$50: now also C49.2; no longer C46.2
- net N$51: now also C50.2; no longer C47.2
- net N$52: now also R41.1; no longer R38.1
- net N$53: now also R40.1; no longer R37.1
- net N$54: now also R37.1; no longer R34.1
- net N$56: now also C62.2; no longer C59.2
- net N$57: now also C61.2; no longer C58.2
- net N$59: now also R35.2; no longer R32.2
- net N$60: now also C63.1, C64.1, RTS3.2; no longer C60.2, RTS3.1
- net N$61: now also R46.1; no longer R42.1
- net N$62: now also R53.2; no longer R49.2
- net N$63: now also R54.2; no longer R50.2
- net N$64: now also R54.1; no longer R50.1
- net N$65: now also C65.2; no longer C61.2
- net N$66: now also C66.2; no longer C62.2
- net N$67: now also R52.1; no longer R48.1
- net N$68: now also R51.1; no longer R47.1
- net N$69: now also R48.1; no longer R44.1
- net N$71: now also C78.2; no longer C74.2
- net N$72: now also C77.2; no longer C73.2
- net N$74: now also R46.2; no longer R42.2
- net N$75: now also C79.1, C80.1, RTS4.2; no longer C75.2, RTS4.1
- net N$76: now also R57.1; no longer R52.1
- net N$77: now also R64.2; no longer R59.2
- net N$78: now also R65.2; no longer R60.2
- net N$79: now also R65.1; no longer R60.1
- net N$80: now also C81.2; no longer C76.2
- net N$81: now also C82.2; no longer C77.2
- net N$82: now also R63.1; no longer R58.1
- net N$83: now also R62.1; no longer R57.1
- net N$84: now also R59.1; no longer R54.1
- net N$86: now also C94.2; no longer C89.2
- net N$87: now also C93.2; no longer C88.2
- net N$89: now also R57.2; no longer R52.2
- net N$90: now also C95.1, C96.1, RTS5.2; no longer C90.2, RTS5.1
- net N$91: now also R68.1; no longer R62.1
- net N$92: now also R75.2; no longer R69.2
- net N$93: now also R76.2; no longer R70.2
- net N$94: now also R76.1; no longer R70.1
- net N$95: now also C97.2; no longer C91.2
- net N$96: now also C98.2; no longer C92.2
- net N$97: now also R74.1; no longer R68.1
- net N$98: now also R73.1; no longer R67.1
- net N$99: now also R70.1; no longer R64.1
- net RXI-0: now also U3.G2; no longer U3.D3
- net RXI-1: now also U9.G2; no longer U9.D3
- net RXI-10: now also U54.G2; no longer U54.D3
- net RXI-11: now also U59.G2; no longer U59.D3
- net RXI-12: now also U64.G2; no longer U64.D3
- net RXI-13: now also U69.G2; no longer U69.D3
- net RXI-14: now also U74.G2; no longer U74.D3
- net RXI-2: now also U14.G2; no longer U14.D3
- net RXI-3: now also U19.G2; no longer U19.D3
- net RXI-4: now also U24.G2; no longer U24.D3
- net RXI-5: now also U29.G2; no longer U29.D3
- net RXI-6: now also U34.G2; no longer U34.D3
- net RXI-7: now also U39.G2; no longer U39.D3
- net RXI-8: now also U44.G2; no longer U44.D3
- net RXI-9: now also U49.G2; no longer U49.D3
- net TXO-0: now also U3.J3; no longer U3.J7
- net TXO-1: now also U9.J3; no longer U9.J7
- net TXO-10: now also U54.J3; no longer U54.J7
- net TXO-11: now also U59.J3; no longer U59.J7
- net TXO-12: now also U64.J3; no longer U64.J7
- net TXO-13: now also U69.J3; no longer U69.J7
- net TXO-14: now also U74.J3; no longer U74.J7
- net TXO-2: now also U14.J3; no longer U14.J7
- net TXO-3: now also U19.J3; no longer U19.J7
- net TXO-4: now also U24.J3; no longer U24.J7
- net TXO-5: now also U29.J3; no longer U29.J7
- net TXO-6: now also U34.J3; no longer U34.J7
- net TXO-7: now also U39.J3; no longer U39.J7
- net TXO-8: now also U44.J3; no longer U44.J7
- net TXO-9: now also U49.J3; no longer U49.J7
- net VIN1: now also C27.1; no longer C26.1
- net VIN10: now also C171.1, R111.2; no longer C161.1, R101.2
- net VIN11: now also C187.1, R122.2; no longer C176.1, R111.2
- net VIN12: now also C203.1, R133.2; no longer C191.1, R121.2
- net VIN13: now also C219.1, R144.2; no longer C206.1, R131.2
- net VIN14: now also C235.1, R155.2; no longer C221.1, R141.2
- net VIN2: now also C43.1, R23.2; no longer C41.1, R21.2
- net VIN3: now also C59.1, R34.2; no longer C56.1, R31.2
- net VIN4: now also C75.1, R45.2; no longer C71.1, R41.2
- net VIN5: now also C91.1, R56.2; no longer C86.1, R51.2
- net VIN6: now also C107.1, R67.2; no longer C101.1, R61.2
- net VIN7: now also C123.1, R78.2; no longer C116.1, R71.2
- net VIN8: now also C139.1, R89.2; no longer C131.1, R81.2
- net VIN9: now also C155.1, R100.2; no longer C146.1, R91.2
- net V_BATT1: now also C26.1; no longer C25.1
- net V_BATT10: now also C170.1; no longer C160.1
- net V_BATT11: now also C186.1; no longer C175.1
- net V_BATT12: now also C202.1; no longer C190.1
- net V_BATT13: now also C218.1; no longer C205.1
- net V_BATT14: now also C234.1; no longer C220.1
- net V_BATT2: now also C42.1; no longer C40.1
- net V_BATT3: now also C58.1; no longer C55.1
- net V_BATT4: now also C74.1; no longer C70.1
- net V_BATT5: now also C90.1; no longer C85.1
- net V_BATT6: now also C106.1; no longer C100.1
- net V_BATT7: now also C122.1; no longer C115.1
- net V_BATT8: now also C138.1; no longer C130.1
- net V_BATT9: now also C154.1; no longer C145.1
- net V_USB1: now also C25.1; no longer C24.1
- net V_USB10: now also C169.1; no longer C159.1
- net V_USB11: now also C185.1; no longer C174.1
- net V_USB12: now also C201.1; no longer C189.1
- net V_USB13: now also C217.1; no longer C204.1
- net V_USB14: now also C233.1; no longer C219.1
- net V_USB2: now also C41.1; no longer C39.1
- net V_USB3: now also C57.1; no longer C54.1
- net V_USB4: now also C73.1; no longer C69.1
- net V_USB5: now also C89.1; no longer C84.1
- net V_USB6: now also C105.1; no longer C99.1
- net V_USB7: now also C121.1; no longer C114.1
- net V_USB8: now also C137.1; no longer C129.1
- net V_USB9: now also C153.1; no longer C144.1
- net ~D18/LED1: now also R19.2; no longer R18.2
- net ~D18/LED10: now also R118.2; no longer R108.2
- net ~D18/LED11: now also R129.2; no longer R118.2
- net ~D18/LED12: now also R140.2; no longer R128.2
- net ~D18/LED13: now also R151.2; no longer R138.2
- net ~D18/LED14: now also R162.2; no longer R148.2
- net ~D18/LED2: now also R30.2; no longer R28.2
- net ~D18/LED3: now also R41.2; no longer R38.2
- net ~D18/LED4: now also R52.2; no longer R48.2
- net ~D18/LED5: now also R63.2; no longer R58.2
- net ~D18/LED6: now also R74.2; no longer R68.2
- net ~D18/LED7: now also R85.2; no longer R78.2
- net ~D18/LED8: now also R96.2; no longer R88.2
- net ~D18/LED9: now also R107.2; no longer R98.2
Routing:
- net BOOT13: track 0.00 -> 22.5 mm, vias 0 -> 2
- net BOOT8: track 0.00 -> 22.5 mm, vias 0 -> 2
- net BOOT10: track 0.00 -> 22.5 mm, vias 0 -> 2
- net BOOT3: track 0.00 -> 22.5 mm, vias 0 -> 2
- net BOOT5: track 0.00 -> 22.5 mm, vias 0 -> 2
- net BOOT12: track 0.00 -> 22.5 mm, vias 0 -> 2
- net BOOT11: track 0.00 -> 22.5 mm, vias 0 -> 2
- net BOOT7: track 0.00 -> 22.5 mm, vias 0 -> 2
- net BOOT6: track 0.00 -> 22.5 mm, vias 0 -> 2
- net BOOT: track 0.00 -> 22.5 mm, vias 0 -> 2
- net BOOT2: track 0.00 -> 22.5 mm, vias 0 -> 2
- net BOOT1: track 0.00 -> 22.5 mm, vias 0 -> 2
- net BOOT14: track 0.00 -> 22.5 mm, vias 0 -> 2
- net BOOT9: track 0.00 -> 22.5 mm, vias 0 -> 2
- net BOOT4: track 0.00 -> 22.5 mm, vias 0 -> 2
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Other:
- board size 130 x 206.5 mm -> 130 x 203.2 mm
- board text added: "v11"
- board text removed: "v10"
